File: hardware/kicad/relay.sch (KiCad schematic (older format))
At the start: 5 parts, among them Q1 BC547, Q2 BC547, U1 HONGFA-176-2823

Commit message: Shakedown
Changed lines of the file:
@@
 AR Path="/63201DC8/631E337E" Ref="Q5"  Part="1"
 AR Path="/6320529C/631E337E" Ref="Q7"  Part="1"
-F 0 "Q1" V 4400 2800 50  0000 L CNN
+F 0 "Q7" V 4400 2800 50  0000 L CNN
 F 1 "BC547" V 4650 3000 50  0000 C CNN
 F 2 "Package_TO_SOT_THT:TO-92_Inline" H 4650 2925 50  0001 L CIN
@@
 AR Path="/63201DC8/631E4680" Ref="R5"  Part="1"
 AR Path="/6320529C/631E4680" Ref="R7"  Part="1"
-F 0 "R1" V 3800 2650 50  0000 C CNN
+F 0 "R7" V 3800 2650 50  0000 C CNN
 F 1 "10K" V 3900 2700 50  0000 C CNN
 F 2 "Resistor_THT:R_Axial_DIN0207_L6.3mm_D2.5mm_P2.54mm_Vertical" V 3830 2700 50  0001 C CNN
@@
 AR Path="/63201DC8/631B86E1" Ref="U6"  Part="1"
 AR Path="/6320529C/631B86E1" Ref="U7"  Part="1"
-F 0 "U1" H 5500 3350 50  0000 C CNN
+F 0 "U7" H 5500 3350 50  0000 C CNN
 F 1 "HONGFA-176-2823" H 4850 3350 50  0000 C CNN
 F 2 "PDJR-connectors:HONGFA-176-2823" H 5250 2750 50  0001 C CNN
@@
 AR Path="/63201DC8/631C80B3" Ref="Q6"  Part="1"
 AR Path="/6320529C/631C80B3" Ref="Q8"  Part="1"
-F 0 "Q2" V 4350 3600 50  0000 L CNN
+F 0 "Q8" V 4350 3600 50  0000 L CNN
 F 1 "BC547" V 4650 3750 50  0000 C CNN
 F 2 "Package_TO_SOT_THT:TO-92_Inline" H 4650 3675 50  0001 L CIN
@@
 AR Path="/63201DC8/631D1169" Ref="R6"  Part="1"
 AR Path="/6320529C/631D1169" Ref="R8"  Part="1"
-F 0 "R2" V 3800 3400 50  0000 C CNN
+F 0 "R8" V 3800 3400 50  0000 C CNN
 F 1 "10K" V 3900 3450 50  0000 C CNN
 F 2 "Resistor_THT:R_Axial_DIN0207_L6.3mm_D2.5mm_P2.54mm_Vertical" V 3830 3450 50  0001 C CNN
