File: hardware/kicad/ROM104.sch (KiCad schematic (older format))
At the start: 22 parts, among them J1 Screw_Terminal_01x12, J2 CAN, SW1 INSTANCE, SW2 BUS, U2 MCP2551-I-P, U3 TMR-1211, U4 Teensy_3.2

Commit message: Shakedown
Parts:
- removed U?: L293, Package_DIP:DIP-16_W7.62mm, symbol Driver_Motor:L293
Changed lines of the file:
@@
 	2000 1700 2000 1800
 Connection ~ 2000 1700
-NoConn ~ 9550 5150
 $Comp
 L Switch:SW_DIP_x08 SW1
@@
 Text Label 9550 5350 0    50   ~ 0
 CH1_LED
+Text Label 9550 5150 0    50   ~ 0
+CH2_LED
 Text Label 8450 5150 2    50   ~ 0
-CH2_LED
-Text Label 8450 5050 2    50   ~ 0
 CH3_LED
 $Sheet
@@
 Text Label 1050 7150 2    50   ~ 0
 CH3_LED
-$Comp
-L Driver_Motor:L293 U?
-U 1 1 631CCE25
-P 4450 4250
-F 0 "U?" H 4450 5431 50  0000 C CNN
-F 1 "L293" H 4450 5340 50  0000 C CNN
-F 2 "Package_DIP:DIP-16_W7.62mm" H 4700 3500 50  0001 L CNN
-F 3 "http://www.ti.com/lit/ds/symlink/l293.pdf" H 4150 4950 50  0001 C CNN
-	1    4450 4250
-	1    0    0    -1
-$EndComp
+NoConn ~ 8450 5050
 $EndSCHEMATC

Commit message: Stuff
Parts:
- added D? (x8): D, symbol Device:D
- added K? (x4): DIPxx-1Cxx-51x, Relay_THT:Relay_StandexMeder_DIP_LowProfile, symbol Relay:DIPxx-1Cxx-51x
- added U? (x2): L293D, Package_DIP:DIP-16_W7.62mm, symbol Driver_Motor:L293D
Connections:
- wire segments 143 -> 203
Other:
- moved on the sheet: D1, D2, D3, D4, R12, R13, R14, R9

Commit message: Stuff
Parts:
- added D13, D14, D15, D16, D17, D18, D19, D20: D, Diode_THT:D_A-405_P2.54mm_Vertical_AnodeUp, symbol Device:D
- D10, D11, D12, D5, D6, D7, D8, D9: renamed from D?; footprint (none) -> Diode_THT:D_A-405_P2.54mm_Vertical_AnodeUp
- gave numbers to parts that had none: 6
Connections:
- net labels added: CH0_EN, CH1_EN, CH2_EN, CH3_EN, RST, SET
- net labels removed: CH0_RST, CH0_SET, CH1_RST, CH1_SET, CH2_RST, CH2_SET, CH3_RST, CH3_SET
- wire segments 203 -> 265
- no-connect marks 7 -> 9
Other:
- moved on the sheet: U1, U5

Commit message: Tweaks
Connections:
- net CH0_EN: now also U5.9 (EN3,4); no longer U1.1 (EN1,2)
- net CH1_EN: now also U5.1 (EN1,2); no longer U1.9 (EN3,4)
- net CH2_EN: now also U1.9 (EN3,4); no longer U5.1 (EN1,2)
- net CH3_EN: now also U1.1 (EN1,2); no longer U5.9 (EN3,4)
- net at J1.1 (Pin_1): now also K1.14; no longer K4.1
- net at J1.10 (Pin_10): now also K4.14; no longer K1.1
- net at J1.11 (Pin_11): now also K4.7, K4.8; no longer K1.14
- net at K1.7, K1.8: now also J1.2 (Pin_2); no longer J1.12 (Pin_12)
- net at J1.4 (Pin_4): now also K2.14; no longer K3.1
- net at J1.5 (Pin_5): now also K2.7, K2.8; no longer K3.14
- net at K3.7, K3.8: now also J1.8 (Pin_8); no longer J1.6 (Pin_6)
- net at K2.1: now also J1.6 (Pin_6); no longer J1.7 (Pin_7)
- new net: J1.12 (Pin_12), K4.1
- new net: J1.3 (Pin_3), K1.1
- new net: J1.7 (Pin_7), K3.14
- new net: J1.9 (Pin_9), K3.1
- no-connect marks 9 -> 11
Changed lines of the file:
@@
 L Connector:Screw_Terminal_01x12 J1
 U 1 1 631D36BE
-P 650 4300
-F 0 "J1" H 568 3475 50  0000 C CNN
-F 1 "Screw_Terminal_01x12" H 568 3566 50  0000 C CNN
-F 2 "TerminalBlock_WAGO:TerminalBlock_WAGO_236-112_1x12_P5.00mm_45Degree" H 650 4300 50  0001 C CNN
-F 3 "~" H 650 4300 50  0001 C CNN
-	1    650  4300
-	-1   0    0    1
+P 650 4200
+F 0 "J1" H 568 3375 50  0000 C CNN
+F 1 "Screw_Terminal_01x12" H 568 3466 50  0000 C CNN
+F 2 "TerminalBlock_WAGO:TerminalBlock_WAGO_236-112_1x12_P5.00mm_45Degree" H 650 4200 50  0001 C CNN
+F 3 "~" H 650 4200 50  0001 C CNN
+	1    650  4200
+	-1   0    0    -1
 $EndComp
 $Comp
@@
 Text Label 900  7350 2    50   ~ 0
 CH3_LED
-NoConn ~ 8450 5050
 $Comp
 L Driver_Motor:L293D U5
@@
 	-1   0    0    1
 $EndComp
-Wire Wire Line
-	850  4200 1800 4200
 $Comp
 L Relay:DIPxx-1Cxx-51x K2
@@
 $EndComp
 Wire Wire Line
-	1600 4100 1600 3800
-Wire Wire Line
-	850  4100 1600 4100
-Wire Wire Line
 	1800 3800 1800 4200
 Wire Wire Line
@@
 $EndComp
 Wire Wire Line
-	1700 4400 1700 4300
-Wire Wire Line
-	1700 4300 850  4300
-Wire Wire Line
 	1600 5000 1600 5100
 Wire Wire Line
@@
 Wire Wire Line
 	1800 5200 1300 5200
-Wire Wire Line
-	850  4400 1400 4400
-Wire Wire Line
-	1400 4400 1400 5100
 Wire Wire Line
 	850  4500 1300 4500
@@
 	1700 2200 1700 2100
 Wire Wire Line
-	1700 2100 1100 2100
-Wire Wire Line
-	1100 2100 1100 3700
+	1700 2100 1050 2100
 $Comp
 L Relay:DIPxx-1Cxx-51x K4
@@
 $EndComp
 Wire Wire Line
-	850  4600 1200 4600
-Wire Wire Line
-	1200 4600 1200 5300
+	850  4600 1100 4600
 Wire Wire Line
 	1200 5300 1700 5300
@@
 Wire Wire Line
 	1600 6100 1100 6100
-Wire Wire Line
-	1100 6100 1100 4700
-Wire Wire Line
-	1100 4700 850  4700
 Wire Wire Line
 	1800 6000 1800 6200
@@
 	3100 4800 3400 4800
 Wire Wire Line
-	850  4000 1350 4000
-Wire Wire Line
-	1350 3100 1350 4000
-Wire Wire Line
-	1250 3900 850  3900
-Wire Wire Line
-	1250 3000 1250 3900
-Wire Wire Line
-	1150 2900 1150 3800
-Wire Wire Line
-	850  3700 1100 3700
-Wire Wire Line
-	850  3800 1150 3800
-Wire Wire Line
 	2100 4400 2100 4300
 Wire Wire Line
@@
 Wire Wire Line
 	3300 4100 3300 6300
+Text Label 5250 5200 0    50   ~ 0
+CH3_EN
+Text Label 5250 4600 0    50   ~ 0
+CH2_EN
+Text Label 5250 3000 0    50   ~ 0
+CH1_EN
 Text Label 5250 2400 0    50   ~ 0
-CH3_EN
-Text Label 5250 3000 0    50   ~ 0
-CH2_EN
-Text Label 5250 4600 0    50   ~ 0
-CH1_EN
-Text Label 5250 5200 0    50   ~ 0
 CH0_EN
 Wire Wire Line
@@
 Text Label 9550 4650 0    50   ~ 0
 RST
+Wire Wire Line
+	850  3800 1050 3800
+Wire Wire Line
+	1050 2100 1050 3800
+Wire Wire Line
+	1150 2900 1150 3700
+Wire Wire Line
+	850  3700 1150 3700
+Wire Wire Line
+	1250 3000 1250 3900
+Wire Wire Line
+	850  3900 1250 3900
+Wire Wire Line
+	850  4100 1350 4100
+Wire Wire Line
+	1350 3100 1350 4100
+Wire Wire Line
+	850  4200 1800 4200
+Wire Wire Line
+	850  4000 1600 4000
+Wire Wire Line
+	1600 4000 1600 3800
+Wire Wire Line
+	1400 4300 850  4300
+Wire Wire Line
+	1400 4300 1400 5100
+Wire Wire Line
+	850  4400 1700 4400
+Wire Wire Line
+	1200 4700 1200 5300
+Wire Wire Line
+	1100 4600 1100 6100
+Wire Wire Line
+	850  4700 1200 4700
+NoConn ~ 8450 4150
+NoConn ~ 9950 3700
 NoConn ~ 9550 4750
 NoConn ~ 9550 4850
+NoConn ~ 8450 5050
 $EndSCHEMATC

Commit message: Stuff
Other:
- moved on the sheet: D1, D10, D11, D12, D13, D14, D15, D16, D17, D18, D19, D2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

Commit message: Tweaks
Parts:
- removed D10, D11, D12, D13, D14, D15, D16, D17, D18, D19, D20, D5, D6, D7, D8, D9: D, Diode_THT:D_A-405_P2.54mm_Vertical_AnodeUp, symbol Device:D

Commit message: Stuff
Changed lines of the file:
@@
 	3450 5200 3450 5700
 Wire Wire Line
-	4200 4800 4200 4700
-Wire Wire Line
-	4400 4800 4400 4700
-Wire Wire Line
-	4150 6900 4150 7000
-Wire Wire Line
 	4150 7000 4350 7000
-Wire Wire Line
-	4350 7000 4350 6900
 Wire Wire Line
 	3550 4800 3550 7000
@@
 Wire Wire Line
 	4100 2800 3650 2800
-Wire Wire Line
-	3650 2800 3650 5000
 Connection ~ 4100 2800
 $Comp
@@
 Connection ~ 4050 5000
 Connection ~ 3650 5000
-Wire Wire Line
-	3650 5000 3650 7200
 Text Label 5600 6100 0    50   ~ 0
 CH3_EN
@@
 Wire Wire Line
 	2450 7000 3450 7000
+Wire Wire Line
+	4200 4700 4200 4800
+Wire Wire Line
+	4400 4700 4400 4800
+Wire Wire Line
+	3650 2800 3650 5000
+Wire Wire Line
+	4350 6900 4350 7000
+Wire Wire Line
+	4150 6900 4150 7000
+Wire Wire Line
+	3650 5000 3650 7200
 $EndSCHEMATC

Commit message: Tweaks
Changed lines of the file:
@@
 U 1 1 631C1A0C
 P 4400 800
-F 0 "R9" H 4350 800 50  0000 R CNN
+F 0 "R9" V 4450 1000 50  0000 R CNN
 F 1 "4K7" V 4400 800 39  0000 C CNN
 F 2 "Resistor_THT:R_Axial_DIN0204_L3.6mm_D1.6mm_P5.08mm_Horizontal" V 4330 800 50  0001 C CNN
@@
 U 1 1 631C329D
 P 4800 800
-F 0 "D1" H 4793 545 50  0000 C CNN
-F 1 "LED" H 4793 636 50  0000 C CNN
+F 0 "D1" H 4900 750 50  0000 C CNN
+F 1 "LED" H 4793 636 50  0001 C CNN
 F 2 "LED_THT:LED_D1.8mm_W3.3mm_H2.4mm" H 4800 800 50  0001 C CNN
 F 3 "~" H 4800 800 50  0001 C CNN
@@
 	4550 800  4650 800
 Wire Wire Line
-	4150 800  4250 800
+	4050 800  4250 800
 Wire Wire Line
 	4950 800  5450 800
@@
 U 1 1 631D6F98
 P 4400 1000
-F 0 "R12" H 4350 1000 50  0000 R CNN
+F 0 "R12" V 4450 1250 50  0000 R CNN
 F 1 "4K7" V 4400 1000 39  0000 C CNN
 F 2 "Resistor_THT:R_Axial_DIN0204_L3.6mm_D1.6mm_P5.08mm_Horizontal" V 4330 1000 50  0001 C CNN
@@
 U 1 1 631D739B
 P 4400 1200
-F 0 "R13" H 4350 1200 50  0000 R CNN
+F 0 "R13" V 4450 1450 50  0000 R CNN
 F 1 "4K7" V 4400 1200 39  0000 C CNN
 F 2 "Resistor_THT:R_Axial_DIN0204_L3.6mm_D1.6mm_P5.08mm_Horizontal" V 4330 1200 50  0001 C CNN
@@
 U 1 1 631D7696
 P 4400 1400
-F 0 "R14" H 4350 1400 50  0000 R CNN
+F 0 "R14" V 4450 1650 50  0000 R CNN
 F 1 "4K7" V 4400 1400 39  0000 C CNN
 F 2 "Resistor_THT:R_Axial_DIN0204_L3.6mm_D1.6mm_P5.08mm_Horizontal" V 4330 1400 50  0001 C CNN
@@
 U 1 1 631D7AEF
 P 4800 1000
-F 0 "D2" H 4793 745 50  0000 C CNN
-F 1 "LED" H 4793 836 50  0000 C CNN
+F 0 "D2" H 4900 950 50  0000 C CNN
+F 1 "LED" H 4793 836 50  0001 C CNN
 F 2 "LED_THT:LED_D1.8mm_W3.3mm_H2.4mm" H 4800 1000 50  0001 C CNN
 F 3 "~" H 4800 1000 50  0001 C CNN
@@
 U 1 1 631D7EE7
 P 4800 1200
-F 0 "D3" H 4793 945 50  0000 C CNN
-F 1 "LED" H 4793 1036 50  0000 C CNN
+F 0 "D3" H 4900 1150 50  0000 C CNN
+F 1 "LED" H 4793 1036 50  0001 C CNN
 F 2 "LED_THT:LED_D1.8mm_W3.3mm_H2.4mm" H 4800 1200 50  0001 C CNN
 F 3 "~" H 4800 1200 50  0001 C CNN
@@
 U 1 1 631D8355
 P 4800 1400
-F 0 "D4" H 4793 1145 50  0000 C CNN
-F 1 "LED" H 4793 1236 50  0000 C CNN
+F 0 "D4" H 4900 1350 50  0000 C CNN
+F 1 "LED" H 4793 1236 50  0001 C CNN
 F 2 "LED_THT:LED_D1.8mm_W3.3mm_H2.4mm" H 4800 1400 50  0001 C CNN
 F 3 "~" H 4800 1400 50  0001 C CNN
@@
 $EndComp
 Wire Wire Line
-	4150 1000 4250 1000
+	4050 1000 4250 1000
 Wire Wire Line
-	4150 1200 4250 1200
+	4050 1200 4250 1200
 Wire Wire Line
-	4150 1400 4250 1400
-Text Label 4150 800  2    50   ~ 0
+	4050 1400 4250 1400
+Text Label 4050 800  2    50   ~ 0
 CH0_LED
-Text Label 4150 1000 2    50   ~ 0
+Text Label 4050 1000 2    50   ~ 0
 CH1_LED
-Text Label 4150 1200 2    50   ~ 0
+Text Label 4050 1200 2    50   ~ 0
 CH2_LED
-Text Label 4150 1400 2    50   ~ 0
+Text Label 4050 1400 2    50   ~ 0
 CH3_LED
 $Comp
