File: hardware/kicad/ROM104.kicad_pcb (KiCad board)
At the start: 2 copper layers, 75 x 75 mm, 43 parts, among them J1 Screw_Terminal_01x12, J2 CAN, Q1 BC547, Q2 BC547, Q3 BC547, Q4 BC547, Q5 BC547, Q6 BC547, Q7 BC547, Q8 BC547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

Commit message: Shakedown
Parts:
- moved R14 5.19 mm to (199.7, 117.1), turned to 270 degrees
- moved R13 4.83 mm to (201.9, 114.8), turned to 270 degrees
- moved R12 0.13 mm to (204.0, 117.1)
Connections:
- U4 pad 24: /CH3_LED -> Net-(U4-Pad24)
- U4 pad 25: /CH2_LED -> /CH3_LED
- U4 pad 4: Net-(U4-Pad4) -> /CH2_LED
Routing:
- net /CH3_LED: track 18.4 -> 7.02 mm
- net Net-(D4-Pad2): track 29.4 -> 23.8 mm
- net /CH2_LED: track 12.5 -> 7.22 mm
- net Net-(D3-Pad2): track 24.2 -> 20.1 mm
- net Net-(Q7-Pad1): track 21.5 -> 19.5 mm
- net /CH2_RST: track 45.8 -> 44.2 mm
- net /CH3_SET: track 35.0 -> 33.4 mm
- net /CH1_SET: track 64.3 -> 62.7 mm
- net /CH2_SET: track 49.5 -> 48.0 mm
- net /CH1_RST: track 61.1 -> 59.5 mm
- net /CH0_SET: track 79.1 -> 77.5 mm
- net /CH0_RST: track 75.3 -> 73.7 mm
- net /CH3_RST: track 31.0 -> 29.4 mm
- net GND: vias 19 -> 18

Commit message: Stuff
Parts:
- removed Q1, Q2, Q3, Q4, Q5, Q6, Q7, Q8: BC547, Package_TO_SOT_THT:TO-92_Inline
- removed R1, R2, R3, R4, R5, R6, R7, R8: 10K, Resistor_THT:R_Axial_DIN0207_L6.3mm_D2.5mm_P2.54mm_Vertical
- removed U6, U7: HONGFA-176-2823, PDJR-connectors:HONGFA-176-2823
- added D10: D, Diode_THT:D_A-405_P2.54mm_Vertical_AnodeUp, F.Cu at (67.3, 124.0)
- added D11: D, Diode_THT:D_A-405_P2.54mm_Vertical_AnodeUp, F.Cu at (98.9, 112.7)
- added D12: D, Diode_THT:D_A-405_P2.54mm_Vertical_AnodeUp, F.Cu at (77.2, 124.0)
- added D13: D, Diode_THT:D_A-405_P2.54mm_Vertical_AnodeUp, F.Cu at (87.2, 118.1)
- added D14: D, Diode_THT:D_A-405_P2.54mm_Vertical_AnodeUp, F.Cu at (87.2, 123.6)
- added D15: D, Diode_THT:D_A-405_P2.54mm_Vertical_AnodeUp, F.Cu at (108.9, 112.7)
- added D16: D, Diode_THT:D_A-405_P2.54mm_Vertical_AnodeUp, F.Cu at (77.2, 113.1)
- added D17: D, Diode_THT:D_A-405_P2.54mm_Vertical_AnodeUp, F.Cu at (170.7, 126.2)
- added D18: D, Diode_THT:D_A-405_P2.54mm_Vertical_AnodeUp, F.Cu at (170.7, 131.7)
- added D19: D, Diode_THT:D_A-405_P2.54mm_Vertical_AnodeUp, F.Cu at (155.8, 126.2)
- added D20: D, Diode_THT:D_A-405_P2.54mm_Vertical_AnodeUp, F.Cu at (155.8, 131.7)
- added D5: D, Diode_THT:D_A-405_P2.54mm_Vertical_AnodeUp, F.Cu at (97.2, 118.1)
- added D6: D, Diode_THT:D_A-405_P2.54mm_Vertical_AnodeUp, F.Cu at (67.3, 113.1)
- added D7: D, Diode_THT:D_A-405_P2.54mm_Vertical_AnodeUp, F.Cu at (67.3, 118.6)
- added D8: D, Diode_THT:D_A-405_P2.54mm_Vertical_AnodeUp, F.Cu at (89.0, 112.7)
- added D9: D, Diode_THT:D_A-405_P2.54mm_Vertical_AnodeUp, F.Cu at (77.2, 118.6)
- added K1: DIPxx-1Cxx-51x, Relay_THT:Relay_StandexMeder_DIP_LowProfile, F.Cu at (198.0, 142.5)
- added K2: DIPxx-1Cxx-51x, Relay_THT:Relay_StandexMeder_DIP_LowProfile, F.Cu at (182.9, 142.5)
- added K3: DIPxx-1Cxx-51x, Relay_THT:Relay_StandexMeder_DIP_LowProfile, F.Cu at (167.9, 142.4)
- added K4: DIPxx-1Cxx-51x, Relay_THT:Relay_StandexMeder_DIP_LowProfile, F.Cu at (153.0, 142.4)
- U1, U5: value HONGFA-176-2823 -> L293D; footprint PDJR-connectors:HONGFA-176-2823 -> Package_DIP:DIP-16_W7.62mm
- moved U5 10.4 mm to (168.5, 122.7), turned to 90 degrees
- moved U1 6.66 mm to (145.8, 122.7), turned to 90 degrees
Connections:
- J1 pad 1: /relay00/NO -> Net-(J1-Pad1)
- J1 pad 10: /relay03/NO -> Net-(J1-Pad10)
- J1 pad 11: /relay03/CO -> Net-(J1-Pad11)
- J1 pad 12: /relay03/NC -> Net-(J1-Pad12)
- J1 pad 2: /relay00/CO -> Net-(J1-Pad2)
- J1 pad 3: /relay00/NC -> Net-(J1-Pad3)
- J1 pad 4: /relay01/NO -> Net-(J1-Pad4)
- J1 pad 5: /relay01/CO -> Net-(J1-Pad5)
- J1 pad 6: /relay01/NC -> Net-(J1-Pad6)
- J1 pad 7: /relay02/NO -> Net-(J1-Pad7)
- J1 pad 8: /relay02/CO -> Net-(J1-Pad8)
- J1 pad 9: /relay02/NC -> Net-(J1-Pad9)
- U1 pad 1: +5V -> /CH0_EN
- U1 pad 2: Net-(Q2-Pad1) -> /RST
- U1 pad 4: /relay00/CO -> GND
- U1 pad 5: /relay00/NO -> GND
- U1 pad 6: /relay00/NC -> Net-(D17-Pad2)
- U4 pad 10: /CH2_RST -> /SET
- U4 pad 11: /CH1_SET -> /CH3_EN
- U4 pad 12: /CH1_RST -> /CH2_EN
- U4 pad 13: /CH0_SET -> /CH1_EN
- U4 pad 14: /CH0_RST -> /CH0_EN
- U4 pad 7: /CH3_SET -> Net-(U4-Pad7)
- U4 pad 8: /CH3_RST -> Net-(U4-Pad8)
- U4 pad 9: /CH2_SET -> /RST
- U5 pad 1: +5V -> /CH2_EN
- U5 pad 2: Net-(Q4-Pad1) -> /RST
- U5 pad 4: /relay01/CO -> GND
- U5 pad 5: /relay01/NO -> GND
- U5 pad 6: /relay01/NC -> Net-(D10-Pad1)
Routing:
- net +5V: track 224.9 -> 110.1 mm
- net /CH0_EN: track 0.00 -> 91.0 mm
- net /RST: track 0.00 -> 84.0 mm, vias 0 -> 1
- net /CH0_SET: track 77.5 -> 0.00 mm, vias 1 -> 0
- net /CH0_RST: track 73.7 -> 0.00 mm
- net /CH1_SET: track 62.7 -> 0.00 mm, vias 1 -> 0
- net /CH1_EN: track 0.00 -> 60.4 mm, vias 0 -> 1
- net /CH1_RST: track 59.5 -> 0.00 mm
- net /SET: track 0.00 -> 53.9 mm
- net /relay00/CO: track 51.9 -> 0.00 mm
- net /relay01/CO: track 51.5 -> 0.00 mm
- net /relay02/CO: track 51.1 -> 0.00 mm
- net /relay03/CO: track 50.6 -> 0.00 mm
- net /CH2_EN: track 0.00 -> 50.3 mm
- net /CH2_SET: track 48.0 -> 0.00 mm, vias 1 -> 0
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
Commit message: Tweaks
Parts:
- moved D16 111.5 mm to (187.9, 127.3), turned to 90 degrees
- moved D10 106.5 mm to (172.8, 138.2), turned to 90 degrees
- moved D13 103.8 mm to (187.9, 143.6), turned to 90 degrees
- moved D14 101.7 mm to (187.9, 138.2), turned to 90 degrees
- moved D9 98.8 mm to (172.8, 143.6), turned to 90 degrees
- moved D12 95.6 mm to (172.8, 127.3), turned to 90 degrees
- moved D6 93.9 mm to (157.8, 138.2), turned to 90 degrees
- moved D7 91.6 mm to (157.8, 132.7), turned to 90 degrees
- moved D15 81.5 mm to (187.9, 132.7), turned to 90 degrees
- moved D11 76.5 mm to (172.8, 132.7), turned to 90 degrees
- moved D8 70.4 mm to (157.8, 127.3), turned to 90 degrees
- moved D5 65.7 mm to (157.8, 143.6), turned to 90 degrees
- moved D19 47.5 mm to (202.9, 132.5)
- moved D20 47.2 mm to (202.9, 129.0), turned to 90 degrees
- moved K4 47.1 mm to (200.1, 142.6)
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Connections:
- K1 pad 1: Net-(J1-Pad10) -> Net-(J1-Pad3)
- K1 pad 14: Net-(J1-Pad11) -> Net-(J1-Pad1)
- K1 pad 7: Net-(J1-Pad12) -> Net-(J1-Pad2)
- K1 pad 8: Net-(J1-Pad12) -> Net-(J1-Pad2)
- K2 pad 1: Net-(J1-Pad7) -> Net-(J1-Pad6)
- K2 pad 14: Net-(J1-Pad8) -> Net-(J1-Pad4)
- K2 pad 7: Net-(J1-Pad9) -> Net-(J1-Pad5)
- K2 pad 8: Net-(J1-Pad9) -> Net-(J1-Pad5)
- K3 pad 1: Net-(J1-Pad4) -> Net-(J1-Pad9)
- K3 pad 14: Net-(J1-Pad5) -> Net-(J1-Pad7)
- K3 pad 7: Net-(J1-Pad6) -> Net-(J1-Pad8)
- K3 pad 8: Net-(J1-Pad6) -> Net-(J1-Pad8)
- K4 pad 1: Net-(J1-Pad1) -> Net-(J1-Pad12)
- K4 pad 14: Net-(J1-Pad2) -> Net-(J1-Pad10)
- K4 pad 7: Net-(J1-Pad3) -> Net-(J1-Pad11)
- K4 pad 8: Net-(J1-Pad3) -> Net-(J1-Pad11)
- U1 pad 1: /CH0_EN -> /CH3_EN
- U1 pad 9: /CH1_EN -> /CH2_EN
- U5 pad 1: /CH2_EN -> /CH1_EN
- U5 pad 9: /CH3_EN -> /CH0_EN
Routing:
- net +5V: track 110.1 -> 357.7 mm
- net Net-(J1-Pad8): track 0.00 -> 62.7 mm
- net Net-(J1-Pad5): track 0.00 -> 62.5 mm
- net Net-(J1-Pad2): track 0.00 -> 62.5 mm
- net Net-(J1-Pad11): track 0.00 -> 62.5 mm
- net Net-(D10-Pad1): track 0.00 -> 52.9 mm, vias 0 -> 2
- net Net-(D17-Pad2): track 23.1 -> 63.2 mm, vias 0 -> 2
- net Net-(D19-Pad2): track 13.8 -> 45.9 mm, vias 0 -> 1
- net Net-(D11-Pad2): track 0.00 -> 32.1 mm
- net /SET: track 53.9 -> 84.5 mm, vias 0 -> 5
- net Net-(U4-Pad8): track 28.0 -> 0.00 mm
- net Net-(D5-Pad2): track 0.00 -> 25.3 mm
- net Net-(U4-Pad7): track 21.7 -> 0.00 mm, vias 1 -> 0
- net Net-(J1-Pad6): track 0.00 -> 17.5 mm
- net Net-(J1-Pad7): track 0.00 -> 17.5 mm
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
Commit message: Stuff
Routing:
- net +5V: track 357.7 -> 344.9 mm
- net GND: vias 17 -> 23

Commit message: Tweaks
Parts:
- removed D10, D11, D12, D13, D14, D15, D16, D17, D18, D19, D20, D5, D6, D7, D8, D9: D, Diode_THT:D_A-405_P2.54mm_Vertical_AnodeUp
- moved U5 5.08 mm to (160.3, 112.8)
- moved U1 2.92 mm to (183.9, 112.9)
Routing:
- net +5V: track 344.9 -> 137.0 mm
- net Net-(K4-Pad6): track 45.9 -> 39.0 mm, vias 1 -> 2
- net /RST: track 82.0 -> 88.8 mm
- net /CH3_EN: track 32.5 -> 39.2 mm
- net /SET: track 84.5 -> 91.1 mm
- net /CH0_EN: track 87.2 -> 93.6 mm
- net Net-(K4-Pad2): track 63.2 -> 57.0 mm, vias 2 -> 1
- net /CH1_EN: track 59.7 -> 65.9 mm
- net /CH2_EN: track 63.4 -> 68.2 mm
- net Net-(K3-Pad2): track 30.6 -> 27.4 mm
- net Net-(K1-Pad6): track 14.8 -> 17.9 mm
- net Net-(K1-Pad2): track 25.3 -> 22.4 mm
- net Net-(K2-Pad6): track 32.1 -> 34.4 mm
- net Net-(K2-Pad2): track 52.9 -> 54.6 mm, vias 2 -> 0
- net Net-(J1-Pad8): track 62.7 -> 61.3 mm
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
Commit message: Stuff
Parts:
- added REF**: M2.7, MountingHole:MountingHole_2.7mm_M2.5_Pad, F.Cu at (200.0, 98.0)
Routing:
- net /CH3_EN: track 39.2 -> 36.5 mm
- net /CH2_EN: track 68.2 -> 66.3 mm
- net /SET: track 91.1 -> 89.4 mm
- net /RST: track 88.8 -> 87.2 mm
- net /CH1_EN: track 65.9 -> 64.9 mm

Commit message: Tweaks
Routing:
- net Net-(K1-Pad2): track 22.4 -> 23.9 mm
- net Net-(K2-Pad2): track 54.6 -> 56.0 mm
- net Net-(K2-Pad6): track 34.4 -> 35.7 mm
- net Net-(K1-Pad6): track 17.9 -> 19.0 mm
- net Net-(K4-Pad6): track 39.0 -> 39.7 mm
- net Net-(K3-Pad6): track 23.6 -> 24.2 mm
- net Net-(K3-Pad2): track 27.4 -> 28.0 mm
- net GND: vias 21 -> 22

Commit message: |
Parts:
- moved SW2 2.30 mm to (168.1, 103.9)
- moved C2 2.05 mm to (170.4, 106.9), turned to 270 degrees
Routing:
- net Net-(F1-Pad1): track 10.8 -> 30.4 mm
- net /TERM_A: track 10.2 -> 0.00 mm
- net /CAN_L: track 27.4 -> 20.1 mm
- net /CAN_SCR: track 11.8 -> 8.02 mm
- net +5V: track 137.0 -> 134.7 mm
- net GND: vias 22 -> 21
