File: hardware/kicad/ROM106-new.kicad_pcb (KiCad board)
At the start: 2 copper layers, 100 x 8 mm, 21 parts, among them J1 Screw_Terminal_01x03, J2 Screw_Terminal_01x03, J4 Screw_Terminal_01x03, J5 Screw_Terminal_01x03, J6 Screw_Terminal_01x03, J7 Screw_Terminal_01x03, K1 PE014F05, K2 PE014F05, K3 PE014F05, K4 PE014F05, K5 PE014F05, K6 PE014F05, U1 L293D, U4 L293D, U5 L293D

Commit message: Refactor
Parts:
- added C2: 100nF, Capacitor_SMD:C_0805_2012Metric, F.Cu at (50.1, 96.5)
- moved J1003 718.2 mm to (11.8, 124.4)
- moved J1005 718.2 mm to (44.2, 124.4)
- moved K1002 718.2 mm to (-3.22, 120.8)
- moved K1004 718.2 mm to (29.2, 120.7)
- moved U1001 718.2 mm to (0.91, 92.8)
- moved U1002 718.2 mm to (33.9, 92.8)
- moved C1001 718.2 mm to (4.34, 98.7)
- moved C1002 718.2 mm to (-22.1, 93.7)
- moved C1003 718.2 mm to (12.7, 94.5)
- moved C1004 718.2 mm to (37.4, 98.7)
- moved C1005 718.2 mm to (45.7, 94.5)
- moved C1006 718.2 mm to (70.4, 98.7)
- moved J1001 718.2 mm to (-20.6, 124.4)
- moved J1002 718.2 mm to (-4.42, 124.4)
- moved J1004 718.2 mm to (28.0, 124.4)
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- renumbered C2 to C1001, C3 to C1002, C4 to C1003, C5 to C1004, C6 to C1005, C7 to C1006, J1 to J1001, J2 to J1002, J4 to J1003, J5 to J1004, J6 to J1005, J7 to J1006, K1 to K1001, K2 to K1002, K3 to K1003, K4 to K1004, K5 to K1005, K6 to K1006, U1 to U1001, U4 to U1002, U5 to U1003
Connections:
- net /D16 renamed /D5
- net /D17 renamed /D6
- U1001 pad 1: /D20 -> /D22
- U1001 pad 10: /D22 -> /D9
- U1001 pad 15: /D23 -> /D8
- U1001 pad 2: /D22 -> /D9
- U1001 pad 7: /D23 -> /D8
- U1001 pad 9: /D21 -> /D23
- U1002 pad 1: /D18 -> /D20
- U1002 pad 10: /D22 -> /D9
- U1002 pad 15: /D23 -> /D8
- U1002 pad 2: /D22 -> /D9
- U1002 pad 7: /D23 -> /D8
- U1002 pad 9: /D19 -> /D21
- U1003 pad 10: /D22 -> /D9
- U1003 pad 15: /D23 -> /D8
- U1003 pad 2: /D22 -> /D9
- U1003 pad 7: /D23 -> /D8
Routing:
- net /D9: track 0.00 -> 116.3 mm, vias 0 -> 6
- net /D8: track 0.00 -> 109.5 mm, vias 0 -> 5
- net /D23: track 105.4 -> 11.5 mm, vias 5 -> 0
- net /D22: track 109.5 -> 31.6 mm, vias 6 -> 1
- net /D21: track 61.5 -> 26.9 mm, vias 2 -> 3
- net /D20: track 34.0 -> 4.66 mm, vias 2 -> 0
- net /D19: track 28.9 -> 0.00 mm, vias 4 -> 0
- net +5V: track 176.9 -> 187.6 mm
- net (no net): track 0.00 -> 8.92 mm
- net /D5: track 33.9 -> 28.5 mm, vias 1 -> 0
- net /D6: track 23.4 -> 18.4 mm, vias 3 -> 2
- net /D18: track 0.72 -> 0.00 mm
Other:
- board outline removed
